Commit message: robot coloring and controlling by gazebo

File: diff_bot/urdf/caster_wheel.xacro (robot description, xacro)
@@ -21,5 +21,5 @@
     </link>
     <!-- Caster Wheel Joit -->
-    <joint name="caster_wheel_join" type="fixed">
+    <joint name="caster_wheel_joint" type="fixed">
         <origin xyz="${caster_wheel_offset_x} 0.0 ${caster_wheel_offset_z}" rpy="0.0 0.0 0.0"/>
         <parent link="chassis_link"/>
@@ -40,3 +40,7 @@
         <child link="caster_holder"/>
     </joint>
+    <gazebo reference="caster_wheel_link">
+        <mu1 value="0.001"/>
+        <mu2 value="0.001"/>
+    </gazebo>
 </robot>

File: diff_bot/urdf/chassis.xacro (robot description, xacro)
@@ -23,3 +23,6 @@
         <origin xyz="-${wheel_offset_x} 0.0 0.0"/>
     </joint>
+    <gazebo reference="chassis_link">
+        <material> Gazebo/Grey </material>
+    </gazebo>
 </robot>

File: diff_bot/urdf/properties.xacro (robot description, xacro)
@@ -3,11 +3,11 @@
                                 <!-- Properties -->
     <!-- Chassis -->
-    <xacro:property name="chassis_length" value="0.4"/>
-    <xacro:property name="chassis_width" value="0.3"/>
+    <xacro:property name="chassis_length" value="0.18"/>
+    <xacro:property name="chassis_width" value="0.18"/>
     <xacro:property name="chassis_height" value="0.11"/>
-    <xacro:property name="chassis_mass" value="2.0"/>
+    <xacro:property name="chassis_mass" value="1.0"/>
     <!-- Wheels -->
-    <xacro:property name="wheel_offset_x" value="0.1285"/>
-    <xacro:property name="wheel_offset_y" value="0.112"/>
+    <xacro:property name="wheel_offset_x" value="0.04"/>
+    <xacro:property name="wheel_offset_y" value="0.09"/>
     <xacro:property name="wheel_offset_z" value="-0.025"/>
     <xacro:property name="wheel_thickness" value="0.027"/>
@@ -17,6 +17,6 @@
     <xacro:property name="caster_wheel_radius" value="0.01"/>
     <xacro:property name="caster_wheel_mass" value="0.01"/>
-    <xacro:property name="caster_wheel_offset_x" value="0.370"/>
-    <xacro:property name="caster_wheel_offset_z" value="-0.045"/>
+    <xacro:property name="caster_wheel_offset_x" value="0.150"/>
+    <xacro:property name="caster_wheel_offset_z" value="-0.035"/>
                                 <!-- Colors -->
     <material name="white">

File: diff_bot/urdf/robot.urdf.xacro (robot description, xacro)
@@ -6,4 +6,5 @@
     <xacro:include filename="wheels.xacro"/>
     <xacro:include filename="caster_wheel.xacro"/>
+    <xacro:include filename="gazebo_control.xacro"/>
     <!-- Base Link -->
     <link name="base_link"/>

File: diff_bot/urdf/wheels.xacro (robot description, xacro)
@@ -21,7 +21,7 @@
     </xacro:macro>
     <!-- Wheel Joint Macro -->
-    <xacro:macro name="wheel_joint" params="joint_name wheel_name y_offset roll">
+    <xacro:macro name="wheel_joint" params="joint_name wheel_name y_offset ">
         <joint name="${joint_name}" type="continuous">
-            <origin xyz="0 ${y_offset} 0" rpy="${roll} 0.0 0.0"/>
+            <origin xyz="0 ${y_offset} 0" rpy="${-pi/2} 0.0 0.0"/>
             <parent link="base_link"/>
             <child link="${wheel_name}"/>
@@ -32,8 +32,14 @@
     <xacro:wheel_link link_name="left_wheel_link" />
     <!-- Left Wheel Joint -->
-    <xacro:wheel_joint joint_name="left_wheel_joint" wheel_name="left_wheel_link" y_offset="${wheel_offset_y}" roll="${-pi/2}"/>
+    <xacro:wheel_joint joint_name="left_wheel_joint" wheel_name="left_wheel_link" y_offset="${wheel_offset_y}"/>
     <!-- Right Wheel Link -->
     <xacro:wheel_link link_name="right_wheel_link" />
     <!-- Right Wheel Joint -->
-    <xacro:wheel_joint joint_name="right_wheel_joint" wheel_name="right_wheel_link" y_offset="${-wheel_offset_y}" roll="${pi/2}"/>
+    <xacro:wheel_joint joint_name="right_wheel_joint" wheel_name="right_wheel_link" y_offset="${-wheel_offset_y}"/>
+    <gazebo reference="left_wheel_link">
+        <material> Gazebo/Black </material>
+    </gazebo>
+    <gazebo reference="right_wheel_link">
+        <material> Gazebo/Black </material>
+    </gazebo>
 </robot>
