Commit message: adding control to real robot

File: diff_bot/urdf/properties.xacro (robot description, xacro)
@@ -3,20 +3,20 @@
                                 <!-- Properties -->
     <!-- Chassis -->
-    <xacro:property name="chassis_length" value="0.18"/>
-    <xacro:property name="chassis_width" value="0.18"/>
-    <xacro:property name="chassis_height" value="0.11"/>
+    <xacro:property name="chassis_length" value="0.172"/>
+    <xacro:property name="chassis_width" value="0.156"/>
+    <xacro:property name="chassis_height" value="0.141"/>
     <xacro:property name="chassis_mass" value="1.0"/>
     <!-- Wheels -->
-    <xacro:property name="wheel_offset_x" value="0.04"/>
-    <xacro:property name="wheel_offset_y" value="0.09"/>
-    <xacro:property name="wheel_offset_z" value="-0.025"/>
+    <xacro:property name="wheel_offset_x" value="0.07"/>
+    <xacro:property name="wheel_offset_y" value="0.078"/>
+    <xacro:property name="wheel_offset_z" value="-0.05"/>
     <xacro:property name="wheel_thickness" value="0.027"/>
-    <xacro:property name="wheel_radius" value="0.0325"/>
+    <xacro:property name="wheel_radius" value="0.034"/>
     <xacro:property name="wheel_mass" value="0.037"/>
     <!-- Caster Wheel -->
     <xacro:property name="caster_wheel_radius" value="0.01"/>
     <xacro:property name="caster_wheel_mass" value="0.01"/>
-    <xacro:property name="caster_wheel_offset_x" value="0.150"/>
-    <xacro:property name="caster_wheel_offset_z" value="-0.035"/>
+    <xacro:property name="caster_wheel_offset_x" value="0.162"/>
+    <xacro:property name="caster_wheel_offset_z" value="-0.025"/>
                                 <!-- Colors -->
     <material name="white">

File: diff_bot/urdf/robot.urdf.xacro (robot description, xacro)
@@ -7,4 +7,5 @@
     <xacro:include filename="caster_wheel.xacro"/>
     <xacro:include filename="gazebo_control.xacro"/>
+    <xacro:include filename="control.xacro"/>
     <!-- Base Link -->
     <link name="base_link"/>

Commit message: adding lidar and create first world

File: diff_bot/urdf/properties.xacro (robot description, xacro)
@@ -5,5 +5,5 @@
     <xacro:property name="chassis_length" value="0.172"/>
     <xacro:property name="chassis_width" value="0.156"/>
-    <xacro:property name="chassis_height" value="0.141"/>
+    <xacro:property name="chassis_height" value="0.096"/>
     <xacro:property name="chassis_mass" value="1.0"/>
     <!-- Wheels -->
@@ -19,4 +19,9 @@
     <xacro:property name="caster_wheel_offset_x" value="0.162"/>
     <xacro:property name="caster_wheel_offset_z" value="-0.025"/>
+    <!-- Back Caster Wheel -->
+    <xacro:property name="bcaster_wheel_radius" value="0.01"/>
+    <xacro:property name="bcaster_wheel_mass" value="0.01"/>
+    <xacro:property name="bcaster_wheel_offset_x" value="0.0"/>
+    <xacro:property name="bcaster_wheel_offset_z" value="-0.02"/>
                                 <!-- Colors -->
     <material name="white">

File: diff_bot/urdf/robot.urdf.xacro (robot description, xacro)
@@ -6,6 +6,8 @@
     <xacro:include filename="wheels.xacro"/>
     <xacro:include filename="caster_wheel.xacro"/>
+    <xacro:include filename="bcaster_wheel.xacro"/>
     <xacro:include filename="gazebo_control.xacro"/>
     <xacro:include filename="control.xacro"/>
+    <xacro:include filename="lidar.xacro"/>
     <!-- Base Link -->
     <link name="base_link"/>
