Commit message: first commit

File: diff_bot/urdf/robot.urdf.xacro (robot description, xacro)
@@ -12,3 +12,9 @@
     <!-- Base Link -->
     <link name="base_link"/>
+    <!-- Base Footprint Link -->
+    <link name="base_footprint"/>
+    <joint name="base_footprint_joint" type="fixed">
+        <parent link="base_link"/>
+        <child link="base_footprint"/>
+    </joint>
 </robot>
